File: AE-2U-Protoboard/KiCad/AE-2U-Protoboard.kicad_pcb (KiCad board)
At the start: 2 copper layers, 25 x 100 mm, 336 parts

Commit message: created AE-2U-Protoboard
Parts:
- removed the REF** at (85.1, 37.1)
- removed the REF** at (95.2, 136.2)
- removed the REF** at (105.4, 131.1)
- removed the REF** at (105.4, 37.1)
- removed the REF** at (85.1, 131.1)
- added ?: , , F.Cu at (105.1, 145.1)
- added ?: , , F.Cu at (105.1, 51.1)
- added ? (x2): , , F.Cu at (94.9, 51.0)
- added ?: , , F.Cu at (107.6, 51.1)
- added ?: , , F.Cu at (110.2, 145.1)
- added ?: , , F.Cu at (120.3, 145.2)
- added ? (x2): , , F.Cu at (94.9, 145.2)
- added ?: , , F.Cu at (107.6, 142.6)
- added ?: , , F.Cu at (120.3, 51.0)
- added ?: , , F.Cu at (110.2, 51.1)
- added ?: , , F.Cu at (107.6, 145.1)
- added ?: , , F.Cu at (107.6, 53.7)
- added REF**: Pad, clectric-diy:Pad, F.Cu at (122.8, 61.3)
- added REF**: Pad, clectric-diy:Pad, F.Cu at (84.8, 79.1)
- added REF**: Pad, clectric-diy:Pad, F.Cu at (92.4, 61.3)
- added REF**: Pad, clectric-diy:Pad, F.Cu at (94.9, 107.0)
- added REF**: Pad, clectric-diy:Pad, F.Cu at (120.3, 96.9)
- added REF**: Pad, clectric-diy:Pad, F.Cu at (87.3, 137.5)
- added REF**: Pad, clectric-diy:Pad, F.Cu at (87.3, 132.4)
- added REF**: Pad, clectric-diy:Pad, F.Cu at (89.8, 84.2)
- added REF**: Pad, clectric-diy:Pad, F.Cu at (87.3, 94.3)
- added REF**: Pad, clectric-diy:Pad, F.Cu at (89.8, 61.3)
- added REF**: Pad, clectric-diy:Pad, F.Cu at (84.8, 140.1)
- added REF**: Pad, clectric-diy:Pad, F.Cu at (120.3, 76.5)
- added REF**: Pad, clectric-diy:Pad, F.Cu at (130.5, 137.5)
- added REF**: Pad, clectric-diy:Pad, F.Cu at (127.9, 89.2)
- added REF**: Pad, clectric-diy:Pad, F.Cu at (120.3, 63.9)
- added REF**: Pad, clectric-diy:Pad, F.Cu at (127.9, 51.1)
- added REF**: Pad, clectric-diy:Pad, F.Cu at (84.8, 96.9)
- added REF**: Pad, clectric-diy:Pad, F.Cu at (87.3, 102.0)
- added REF**: Pad, clectric-diy:Pad, F.Cu at (130.5, 127.3)
- added REF**: Pad, clectric-diy:Pad, F.Cu at (94.9, 86.7)
- added REF**: Pad, clectric-diy:Pad, F.Cu at (130.5, 96.9)
- added REF**: Pad, clectric-diy:Pad, F.Cu at (84.8, 84.2)
- added REF**: Pad, clectric-diy:Pad, F.Cu at (125.4, 66.4)
- added REF**: Pad, clectric-diy:Pad, F.Cu at (122.8, 58.8)
- added REF**: Pad, clectric-diy:Pad, F.Cu at (130.5, 122.3)
- added REF**: Pad, clectric-diy:Pad, F.Cu at (87.3, 51.1)
- added REF**: Pad, clectric-diy:Pad, F.Cu at (107.6, 145.1)
- added REF**: Pad, clectric-diy:Pad, F.Cu at (127.9, 145.1)
- added REF**: Pad, clectric-diy:Pad, F.Cu at (84.8, 122.3)
- added REF**: Pad, clectric-diy:Pad, F.Cu at (127.9, 142.6)
- added REF**: Pad, clectric-diy:Pad, F.Cu at (92.4, 109.6)
- added REF**: Pad, clectric-diy:Pad, F.Cu at (92.4, 140.1)
- added REF**: Pad, clectric-diy:Pad, F.Cu at (125.4, 63.9)
- added REF**: Pad, clectric-diy:Pad, F.Cu at (87.3, 140.1)
- added REF**: Pad, clectric-diy:Pad, F.Cu at (125.4, 102.0)
- added REF**: Pad, clectric-diy:Pad, F.Cu at (120.3, 71.5)
- added REF**: Pad, clectric-diy:Pad, F.Cu at (92.4, 94.3)
- added REF**: Pad, clectric-diy:Pad, F.Cu at (120.3, 122.3)
- added REF**: Pad, clectric-diy:Pad, F.Cu at (92.4, 63.9)
- added REF**: Pad, clectric-diy:Pad, F.Cu at (130.5, 68.9)
- added REF**: Pad, clectric-diy:Pad, F.Cu at (94.9, 84.2)
- added REF**: Pad, clectric-diy:Pad, F.Cu at (130.5, 53.7)
- added REF**: Pad, clectric-diy:Pad, F.Cu at (92.4, 132.4)
- added REF**: Pad, clectric-diy:Pad, F.Cu at (107.6, 51.1)
- added REF**: Pad, clectric-diy:Pad, F.Cu at (87.3, 112.1)
- added REF**: Pad, clectric-diy:Pad, F.Cu at (120.3, 132.4)
- added REF**: Pad, clectric-diy:Pad, F.Cu at (110.2, 51.1)
- added REF**: Pad, clectric-diy:Pad, F.Cu at (87.3, 114.7)
- added REF**: Pad, clectric-diy:Pad, F.Cu at (89.8, 66.4)
- added REF**: Pad, clectric-diy:Pad, F.Cu at (84.8, 117.2)
- added REF**: Pad, clectric-diy:Pad, F.Cu at (127.9, 86.7)
- added REF**: Pad, clectric-diy:Pad, F.Cu at (89.8, 129.9)
- added REF**: Pad, clectric-diy:Pad, F.Cu at (84.8, 129.9)
- added REF**: Pad, clectric-diy:Pad, F.Cu at (89.8, 91.8)
- added REF**: Pad, clectric-diy:Pad, F.Cu at (120.3, 137.5)
- added REF**: Pad, clectric-diy:Pad, F.Cu at (127.9, 124.8)
- added REF**: Pad, clectric-diy:Pad, F.Cu at (120.3, 114.7)
- added REF**: Pad, clectric-diy:Pad, F.Cu at (92.4, 53.7)
- added REF**: Pad, clectric-diy:Pad, F.Cu at (127.9, 53.7)
- added REF**: Pad, clectric-diy:Pad, F.Cu at (84.8, 86.7)
- added REF**: Pad, clectric-diy:Pad, F.Cu at (84.8, 127.3)
- added REF**: Pad, clectric-diy:Pad, F.Cu at (120.3, 84.2)
- added REF**: Pad, clectric-diy:Pad, F.Cu at (84.8, 137.5)
- added REF**: Pad, clectric-diy:Pad, F.Cu at (89.8, 74.0)
- added REF**: Pad, clectric-diy:Pad, F.Cu at (94.9, 117.2)
- added REF**: Pad, clectric-diy:Pad, F.Cu at (94.9, 71.5)
- added REF**: Pad, clectric-diy:Pad, F.Cu at (89.8, 56.2)
- added REF**: Pad, clectric-diy:Pad, F.Cu at (89.8, 79.1)
- added REF**: Pad, clectric-diy:Pad, F.Cu at (84.8, 53.7)
- added REF**: Pad, clectric-diy:Pad, F.Cu at (127.9, 79.1)
- added REF**: Pad, clectric-diy:Pad, F.Cu at (122.8, 135.0)
- added REF**: Pad, clectric-diy:Pad, F.Cu at (120.3, 129.9)
- added REF**: Pad, clectric-diy:Pad, F.Cu at (89.8, 107.0)
- added REF**: Pad, clectric-diy:Pad, F.Cu at (89.8, 114.7)
- added REF**: Pad, clectric-diy:Pad, F.Cu at (92.4, 79.1)
- added REF**: Pad, clectric-diy:Pad, F.Cu at (127.9, 112.1)
- added REF**: Pad, clectric-diy:Pad, F.Cu at (94.9, 127.3)
- added REF**: Pad, clectric-diy:Pad, F.Cu at (127.9, 114.7)
- added REF**: Pad, clectric-diy:Pad, F.Cu at (127.9, 96.9)
- added REF**: Pad, clectric-diy:Pad, F.Cu at (107.6, 142.6)
- added REF**: Pad, clectric-diy:Pad, F.Cu at (130.5, 119.7)
- added REF**: Pad, clectric-diy:Pad, F.Cu at (130.5, 84.2)
- added REF**: Pad, clectric-diy:Pad, F.Cu at (92.4, 91.8)
- added REF**: Pad, clectric-diy:Pad, F.Cu at (89.8, 76.5)
- added REF**: Pad, clectric-diy:Pad, F.Cu at (92.4, 127.3)
- added REF**: Pad, clectric-diy:Pad, F.Cu at (125.4, 79.1)
- added REF**: Pad, clectric-diy:Pad, F.Cu at (120.3, 61.3)
- added REF**: Pad, clectric-diy:Pad, F.Cu at (125.4, 56.2)
- added REF**: Pad, clectric-diy:Pad, F.Cu at (84.8, 104.5)
- added REF**: Pad, clectric-diy:Pad, F.Cu at (125.4, 76.5)
- added REF**: Pad, clectric-diy:Pad, F.Cu at (127.9, 129.9)
- added REF**: Pad, clectric-diy:Pad, F.Cu at (130.5, 81.6)
- added REF**: Pad, clectric-diy:Pad, F.Cu at (89.8, 109.6)
- added REF**: Pad, clectric-diy:Pad, F.Cu at (84.8, 68.9)
- added REF**: Pad, clectric-diy:Pad, F.Cu at (87.3, 124.8)
- added REF**: Pad, clectric-diy:Pad, F.Cu at (89.8, 63.9)
- added REF**: Pad, clectric-diy:Pad, F.Cu at (127.9, 84.2)
- added REF**: Pad, clectric-diy:Pad, F.Cu at (87.3, 86.7)
- added REF**: Pad, clectric-diy:Pad, F.Cu at (89.8, 68.9)
- added REF**: Pad, clectric-diy:Pad, F.Cu at (87.3, 99.4)
- added REF**: Pad, clectric-diy:Pad, F.Cu at (122.8, 99.4)
- added REF**: Pad, clectric-diy:Pad, F.Cu at (84.8, 135.0)
- added REF**: Pad, clectric-diy:Pad, F.Cu at (84.8, 56.2)
- added REF**: Pad, clectric-diy:Pad, F.Cu at (84.8, 76.5)
- added REF**: Pad, clectric-diy:Pad, F.Cu at (84.8, 119.7)
- added REF**: Pad, clectric-diy:Pad, F.Cu at (130.5, 51.1)
- added REF**: Pad, clectric-diy:Pad, F.Cu at (84.8, 142.6)
- added REF**: Pad, clectric-diy:Pad, F.Cu at (84.8, 124.8)
- added REF**: Pad, clectric-diy:Pad, F.Cu at (125.4, 132.4)
- added REF**: Pad, clectric-diy:Pad, F.Cu at (127.9, 91.8)
- added REF**: Pad, clectric-diy:Pad, F.Cu at (87.3, 129.9)
- added REF**: Pad, clectric-diy:Pad, F.Cu at (84.8, 51.1)
- added REF**: Pad, clectric-diy:Pad, F.Cu at (94.9, 124.8)
- added REF**: Pad, clectric-diy:Pad, F.Cu at (92.4, 122.3)
- added REF**: Pad, clectric-diy:Pad, F.Cu at (120.3, 99.4)
- added REF**: Pad, clectric-diy:Pad, F.Cu at (84.8, 102.0)
- added REF**: Pad, clectric-diy:Pad, F.Cu at (92.4, 99.4)
- added REF**: Pad, clectric-diy:Pad, F.Cu at (87.3, 142.6)
- added REF**: Pad, clectric-diy:Pad, F.Cu at (125.4, 135.0)
- added REF**: Pad, clectric-diy:Pad, F.Cu at (125.4, 61.3)
- added REF**: Pad, clectric-diy:Pad, F.Cu at (84.8, 66.4)
- added REF**: Pad, clectric-diy:Pad, F.Cu at (94.9, 79.1)
- added REF**: Pad, clectric-diy:Pad, F.Cu at (125.4, 89.2)
- added REF**: Pad, clectric-diy:Pad, F.Cu at (87.3, 68.9)
- added REF**: Pad, clectric-diy:Pad, F.Cu at (130.5, 56.2)
- added REF**: Pad, clectric-diy:Pad, F.Cu at (130.5, 94.3)
- added REF**: Pad, clectric-diy:Pad, F.Cu at (92.4, 135.0)
- added REF**: Pad, clectric-diy:Pad, F.Cu at (87.3, 89.2)
- added REF**: Pad, clectric-diy:Pad, F.Cu at (84.8, 114.7)
- added REF**: Pad, clectric-diy:Pad, F.Cu at (87.3, 71.5)
- added REF**: Pad, clectric-diy:Pad, F.Cu at (130.5, 104.5)
- added REF**: Pad, clectric-diy:Pad, F.Cu at (125.4, 91.8)
- added REF**: Pad, clectric-diy:Pad, F.Cu at (127.9, 140.1)
- added REF**: Pad, clectric-diy:Pad, F.Cu at (89.8, 119.7)
- added REF**: Pad, clectric-diy:Pad, F.Cu at (122.8, 76.5)
- added REF**: Pad, clectric-diy:Pad, F.Cu at (94.9, 96.9)
- added REF**: Pad, clectric-diy:Pad, F.Cu at (120.3, 56.2)
- added REF**: Pad, clectric-diy:Pad, F.Cu at (125.4, 84.2)
- added REF**: Pad, clectric-diy:Pad, F.Cu at (84.8, 132.4)
- added REF**: Pad, clectric-diy:Pad, F.Cu at (92.4, 119.7)
- added REF**: Pad, clectric-diy:Pad, F.Cu at (120.3, 74.0)
- added REF**: Pad, clectric-diy:Pad, F.Cu at (107.6, 53.7)
- added REF**: Pad, clectric-diy:Pad, F.Cu at (127.9, 74.0)
- added REF**: Pad, clectric-diy:Pad, F.Cu at (130.5, 66.4)
- added REF**: Pad, clectric-diy:Pad, F.Cu at (87.3, 109.6)
- added REF**: Pad, clectric-diy:Pad, F.Cu at (130.5, 135.0)
- added REF**: Pad, clectric-diy:Pad, F.Cu at (122.8, 119.7)
- added REF**: Pad, clectric-diy:Pad, F.Cu at (120.3, 107.0)
- added REF**: Pad, clectric-diy:Pad, F.Cu at (89.8, 102.0)
- added REF**: Pad, clectric-diy:Pad, F.Cu at (125.4, 109.6)
- added REF**: Pad, clectric-diy:Pad, F.Cu at (87.3, 66.4)
- added REF**: Pad, clectric-diy:Pad, F.Cu at (94.9, 112.1)
- added REF**: Pad, clectric-diy:Pad, F.Cu at (122.8, 107.0)
- added REF**: Pad, clectric-diy:Pad, F.Cu at (122.8, 84.2)
- added REF**: Pad, clectric-diy:Pad, F.Cu at (125.4, 68.9)
- added REF**: Pad, clectric-diy:Pad, F.Cu at (122.8, 94.3)
- added REF**: Pad, clectric-diy:Pad, F.Cu at (127.9, 137.5)
- added REF**: Pad, clectric-diy:Pad, F.Cu at (92.4, 84.2)
- added REF**: Pad, clectric-diy:Pad, F.Cu at (84.8, 145.1)
- added REF**: Pad, clectric-diy:Pad, F.Cu at (130.5, 145.1)
- added REF**: Pad, clectric-diy:Pad, F.Cu at (92.4, 117.2)
- added REF**: Pad, clectric-diy:Pad, F.Cu at (125.4, 96.9)
- added REF**: Pad, clectric-diy:Pad, F.Cu at (94.9, 76.5)
- added REF**: Pad, clectric-diy:Pad, F.Cu at (127.9, 76.5)
- added REF**: Pad, clectric-diy:Pad, F.Cu at (125.4, 114.7)
- added REF**: Pad, clectric-diy:Pad, F.Cu at (122.8, 53.7)
- added REF**: Pad, clectric-diy:Pad, F.Cu at (122.8, 122.3)
- added REF**: Pad, clectric-diy:Pad, F.Cu at (125.4, 124.8)
- added REF**: Pad, clectric-diy:Pad, F.Cu at (120.3, 89.2)
- added REF**: Pad, clectric-diy:Pad, F.Cu at (125.4, 71.5)
- added REF**: Pad, clectric-diy:Pad, F.Cu at (89.8, 124.8)
- added REF**: Pad, clectric-diy:Pad, F.Cu at (87.3, 135.0)
- added REF**: Pad, clectric-diy:Pad, F.Cu at (130.5, 114.7)
- added REF**: Pad, clectric-diy:Pad, F.Cu at (130.5, 142.6)
- added REF**: Pad, clectric-diy:Pad, F.Cu at (89.8, 104.5)
- added REF**: Pad, clectric-diy:Pad, F.Cu at (94.9, 132.4)
- added REF**: Pad, clectric-diy:Pad, F.Cu at (122.8, 127.3)
- added REF**: Pad, clectric-diy:Pad, F.Cu at (94.9, 102.0)
- added REF**: Pad, clectric-diy:Pad, F.Cu at (84.8, 61.3)
- added REF**: Pad, clectric-diy:Pad, F.Cu at (122.8, 86.7)
- added REF**: Pad, clectric-diy:Pad, F.Cu at (92.4, 137.5)
- added REF**: Pad, clectric-diy:Pad, F.Cu at (94.9, 104.5)
- added REF**: Pad, clectric-diy:Pad, F.Cu at (87.3, 58.8)
- added REF**: Pad, clectric-diy:Pad, F.Cu at (127.9, 127.3)
- added REF**: Pad, clectric-diy:Pad, F.Cu at (127.9, 66.4)
- added REF**: Pad, clectric-diy:Pad, F.Cu at (94.9, 74.0)
- added REF**: Pad, clectric-diy:Pad, F.Cu at (89.8, 71.5)
- added REF**: Pad, clectric-diy:Pad, F.Cu at (94.9, 94.3)
- added REF**: Pad, clectric-diy:Pad, F.Cu at (130.5, 63.9)
- added REF**: Pad, clectric-diy:Pad, F.Cu at (125.4, 51.1)
- added REF**: Pad, clectric-diy:Pad, F.Cu at (120.3, 102.0)
- added REF**: Pad, clectric-diy:Pad, F.Cu at (125.4, 127.3)
- added REF**: Pad, clectric-diy:Pad, F.Cu at (92.4, 96.9)
- added REF**: Pad, clectric-diy:Pad, F.Cu at (89.8, 94.3)
- added REF**: Pad, clectric-diy:Pad, F.Cu at (105.1, 145.1)
- added REF**: Pad, clectric-diy:Pad, F.Cu at (122.8, 66.4)
- added REF**: Pad, clectric-diy:Pad, F.Cu at (125.4, 99.4)
- added REF**: Pad, clectric-diy:Pad, F.Cu at (120.3, 135.0)
- added REF**: Pad, clectric-diy:Pad, F.Cu at (125.4, 81.6)
- added REF**: Pad, clectric-diy:Pad, F.Cu at (89.8, 51.1)
- added REF**: Pad, clectric-diy:Pad, F.Cu at (89.8, 142.6)
- added REF**: Pad, clectric-diy:Pad, F.Cu at (94.9, 58.8)
- added REF**: Pad, clectric-diy:Pad, F.Cu at (84.8, 74.0)
- added REF**: Pad, clectric-diy:Pad, F.Cu at (122.8, 79.1)
- added REF**: Pad, clectric-diy:Pad, F.Cu at (130.5, 124.8)
- added REF**: Pad, clectric-diy:Pad, F.Cu at (94.9, 114.7)
- added REF**: Pad, clectric-diy:Pad, F.Cu at (87.3, 63.9)
- added REF**: Pad, clectric-diy:Pad, F.Cu at (84.8, 109.6)
- added REF**: Pad, clectric-diy:Pad, F.Cu at (120.3, 79.1)
- added REF**: Pad, clectric-diy:Pad, F.Cu at (125.4, 74.0)
- added REF**: Pad, clectric-diy:Pad, F.Cu at (125.4, 53.7)
- added REF**: Pad, clectric-diy:Pad, F.Cu at (89.8, 145.1)
- added REF**: Pad, clectric-diy:Pad, F.Cu at (94.9, 129.9)
- added REF**: Pad, clectric-diy:Pad, F.Cu at (87.3, 145.1)
- added REF**: Pad, clectric-diy:Pad, F.Cu at (84.8, 63.9)
- added REF**: Pad, clectric-diy:Pad, F.Cu at (130.5, 89.2)
- added REF**: Pad, clectric-diy:Pad, F.Cu at (125.4, 129.9)
- added REF**: Pad, clectric-diy:Pad, F.Cu at (92.4, 102.0)
- added REF**: Pad, clectric-diy:Pad, F.Cu at (130.5, 99.4)
- added REF**: Pad, clectric-diy:Pad, F.Cu at (92.4, 89.2)
- added REF**: Pad, clectric-diy:Pad, F.Cu at (125.4, 137.5)
- added REF**: Pad, clectric-diy:Pad, F.Cu at (122.8, 71.5)
- added REF**: Pad, clectric-diy:Pad, F.Cu at (92.4, 142.6)
- added REF**: Pad, clectric-diy:Pad, F.Cu at (120.3, 66.4)
- added REF**: Pad, clectric-diy:Pad, F.Cu at (87.3, 122.3)
- added REF**: Pad, clectric-diy:Pad, F.Cu at (125.4, 104.5)
- added REF**: Pad, clectric-diy:Pad, F.Cu at (92.4, 124.8)
- added REF**: Pad, clectric-diy:Pad, F.Cu at (92.4, 71.5)
- added REF**: Pad, clectric-diy:Pad, F.Cu at (122.8, 68.9)
- added REF**: Pad, clectric-diy:Pad, F.Cu at (84.8, 99.4)
- added REF**: Pad, clectric-diy:Pad, F.Cu at (94.9, 68.9)
- added REF**: Pad, clectric-diy:Pad, F.Cu at (127.9, 117.2)
- added REF**: Pad, clectric-diy:Pad, F.Cu at (125.4, 145.1)
- added REF**: Pad, clectric-diy:Pad, F.Cu at (122.8, 104.5)
- added REF**: Pad, clectric-diy:Pad, F.Cu at (87.3, 56.2)
- added REF**: Pad, clectric-diy:Pad, F.Cu at (122.8, 142.6)
- added REF**: Pad, clectric-diy:Pad, F.Cu at (125.4, 140.1)
- added REF**: Pad, clectric-diy:Pad, F.Cu at (127.9, 56.2)
- added REF**: Pad, clectric-diy:Pad, F.Cu at (87.3, 84.2)
- added REF**: Pad, clectric-diy:Pad, F.Cu at (125.4, 86.7)
- added REF**: Pad, clectric-diy:Pad, F.Cu at (92.4, 104.5)
- added REF**: Pad, clectric-diy:Pad, F.Cu at (84.8, 81.6)
- added REF**: Pad, clectric-diy:Pad, F.Cu at (120.3, 119.7)
- added REF**: Pad, clectric-diy:Pad, F.Cu at (120.3, 140.1)
- added REF**: Pad, clectric-diy:Pad, F.Cu at (125.4, 112.1)
- added REF**: Pad, clectric-diy:Pad, F.Cu at (84.8, 71.5)
- added REF**: Pad, clectric-diy:Pad, F.Cu at (130.5, 61.3)
- added REF**: Pad, clectric-diy:Pad, F.Cu at (89.8, 112.1)
- added REF**: Pad, clectric-diy:Pad, F.Cu at (92.4, 86.7)
- added REF**: Pad, clectric-diy:Pad, F.Cu at (127.9, 122.3)
- added REF**: Pad, clectric-diy:Pad, F.Cu at (130.5, 112.1)
- added REF**: Pad, clectric-diy:Pad, F.Cu at (94.9, 140.1)
- added REF**: Pad, clectric-diy:Pad, F.Cu at (89.8, 135.0)
- added REF**: Pad, clectric-diy:Pad, F.Cu at (122.8, 56.2)
- added REF**: Pad, clectric-diy:Pad, F.Cu at (120.3, 117.2)
- added REF**: Pad, clectric-diy:Pad, F.Cu at (87.3, 81.6)
- added REF**: Pad, clectric-diy:Pad, F.Cu at (125.4, 107.0)
- added REF**: Pad, clectric-diy:Pad, F.Cu at (120.3, 68.9)
- added REF**: Pad, clectric-diy:Pad, F.Cu at (120.3, 112.1)
- added REF**: Pad, clectric-diy:Pad, F.Cu at (92.4, 107.0)
- added REF**: Pad, clectric-diy:Pad, F.Cu at (92.4, 129.9)
- added REF**: Pad, clectric-diy:Pad, F.Cu at (130.5, 91.8)
- added REF**: Pad, clectric-diy:Pad, F.Cu at (89.8, 132.4)
- added REF**: Pad, clectric-diy:Pad, F.Cu at (94.9, 56.2)
- added REF**: Pad, clectric-diy:Pad, F.Cu at (87.3, 104.5)
- added REF**: Pad, clectric-diy:Pad, F.Cu at (130.5, 71.5)
- added REF**: Pad, clectric-diy:Pad, F.Cu at (122.8, 74.0)
- added REF**: Pad, clectric-diy:Pad, F.Cu at (94.9, 91.8)
- added REF**: Pad, clectric-diy:Pad, F.Cu at (120.3, 127.3)
- added REF**: Pad, clectric-diy:Pad, F.Cu at (125.4, 122.3)
- added REF**: Pad, clectric-diy:Pad, F.Cu at (89.8, 127.3)
- added REF**: Pad, clectric-diy:Pad, F.Cu at (130.5, 76.5)
- added REF**: Pad, clectric-diy:Pad, F.Cu at (84.8, 58.8)
- added REF**: Pad, clectric-diy:Pad, F.Cu at (87.3, 76.5)
- added REF**: Pad, clectric-diy:Pad, F.Cu at (89.8, 86.7)
- added REF**: Pad, clectric-diy:Pad, F.Cu at (87.3, 117.2)
- added REF**: Pad, clectric-diy:Pad, F.Cu at (87.3, 119.7)
- added REF**: Pad, clectric-diy:Pad, F.Cu at (122.8, 91.8)
- added REF**: Pad, clectric-diy:Pad, F.Cu at (120.3, 86.7)
- added REF**: Pad, clectric-diy:Pad, F.Cu at (127.9, 107.0)
- added REF**: Pad, clectric-diy:Pad, F.Cu at (127.9, 109.6)
- added REF**: Pad, clectric-diy:Pad, F.Cu at (89.8, 99.4)
- added REF**: Pad, clectric-diy:Pad, F.Cu at (127.9, 102.0)
- added REF**: Pad, clectric-diy:Pad, F.Cu at (84.8, 89.2)
- added REF**: Pad, clectric-diy:Pad, F.Cu at (89.8, 122.3)
- added REF**: Pad, clectric-diy:Pad, F.Cu at (84.8, 107.0)
- added REF**: Pad, clectric-diy:Pad, F.Cu at (94.9, 137.5)
- added REF**: Pad, clectric-diy:Pad, F.Cu at (120.3, 91.8)
- added REF**: Pad, clectric-diy:Pad, F.Cu at (94.9, 61.3)
- added REF**: Pad, clectric-diy:Pad, F.Cu at (127.9, 99.4)
- added REF**: Pad, clectric-diy:Pad, F.Cu at (122.8, 96.9)
- added REF**: Pad, clectric-diy:Pad, F.Cu at (127.9, 119.7)
- added REF**: Pad, clectric-diy:Pad, F.Cu at (125.4, 142.6)
- added REF**: Pad, clectric-diy:Pad, F.Cu at (122.8, 124.8)
- added REF**: Pad, clectric-diy:Pad, F.Cu at (92.4, 58.8)
- added REF**: Pad, clectric-diy:Pad, F.Cu at (130.5, 132.4)
- added REF**: Pad, clectric-diy:Pad, F.Cu at (130.5, 86.7)
- added REF**: Pad, clectric-diy:Pad, F.Cu at (127.9, 132.4)
- added REF**: Pad, clectric-diy:Pad, F.Cu at (125.4, 58.8)
- added REF**: Pad, clectric-diy:Pad, F.Cu at (122.8, 81.6)
- added REF**: Pad, clectric-diy:Pad, F.Cu at (130.5, 102.0)
- added REF**: Pad, clectric-diy:Pad, F.Cu at (130.5, 107.0)
- added REF**: Pad, clectric-diy:Pad, F.Cu at (92.4, 66.4)
- added REF**: Pad, clectric-diy:Pad, F.Cu at (120.3, 104.5)
- added REF**: Pad, clectric-diy:Pad, F.Cu at (87.3, 127.3)
- added REF**: Pad, clectric-diy:Pad, F.Cu at (125.4, 119.7)
- added REF**: Pad, clectric-diy:Pad, F.Cu at (130.5, 129.9)
- added REF**: Pad, clectric-diy:Pad, F.Cu at (127.9, 61.3)
- added REF**: Pad, clectric-diy:Pad, F.Cu at (127.9, 94.3)
- added REF**: Pad, clectric-diy:Pad, F.Cu at (122.8, 140.1)
- added REF**: Pad, clectric-diy:Pad, F.Cu at (84.8, 94.3)
- added REF**: Pad, clectric-diy:Pad, F.Cu at (89.8, 140.1)
- added REF**: Pad, clectric-diy:Pad, F.Cu at (122.8, 114.7)
- added REF**: Pad, clectric-diy:Pad, F.Cu at (94.9, 66.4)
- added REF**: Pad, clectric-diy:Pad, F.Cu at (122.8, 89.2)
- added REF**: Pad, clectric-diy:Pad, F.Cu at (89.8, 81.6)
- added REF**: Pad, clectric-diy:Pad, F.Cu at (127.9, 58.8)
- added REF**: Pad, clectric-diy:Pad, F.Cu at (130.5, 74.0)
- added REF**: Pad, clectric-diy:Pad, F.Cu at (127.9, 63.9)
- added REF**: Pad, clectric-diy:Pad, F.Cu at (94.9, 119.7)
- added REF**: Pad, clectric-diy:Pad, F.Cu at (120.3, 109.6)
- added REF**: Pad, clectric-diy:Pad, F.Cu at (120.3, 58.8)
- added REF**: Pad, clectric-diy:Pad, F.Cu at (127.9, 81.6)
- added REF**: Pad, clectric-diy:Pad, F.Cu at (92.4, 81.6)
- added REF**: Pad, clectric-diy:Pad, F.Cu at (87.3, 74.0)
- added REF**: Pad, clectric-diy:Pad, F.Cu at (84.8, 91.8)
- added REF**: Pad, clectric-diy:Pad, F.Cu at (89.8, 53.7)
- added REF**: Pad, clectric-diy:Pad, F.Cu at (120.3, 124.8)
- added REF**: Pad, clectric-diy:Pad, F.Cu at (92.4, 74.0)
- added REF**: Pad, clectric-diy:Pad, F.Cu at (94.9, 89.2)
- added REF**: Pad, clectric-diy:Pad, F.Cu at (92.4, 112.1)
- added REF**: Pad, clectric-diy:Pad, F.Cu at (89.8, 58.8)
- added REF**: Pad, clectric-diy:Pad, F.Cu at (87.3, 53.7)
- added REF**: Pad, clectric-diy:Pad, F.Cu at (122.8, 137.5)
- added REF**: Pad, clectric-diy:Pad, F.Cu at (120.3, 81.6)
- added REF**: Pad, clectric-diy:Pad, F.Cu at (127.9, 68.9)
- added REF**: Pad, clectric-diy:Pad, F.Cu at (87.3, 61.3)
- added REF**: Pad, clectric-diy:Pad, F.Cu at (130.5, 140.1)
- added REF**: Pad, clectric-diy:Pad, F.Cu at (125.4, 94.3)
- added REF**: Pad, clectric-diy:Pad, F.Cu at (127.9, 135.0)
- added REF**: Pad, clectric-diy:Pad, F.Cu at (92.4, 76.5)
- added REF**: Pad, clectric-diy:Pad, F.Cu at (94.9, 122.3)
- added REF**: Pad, clectric-diy:Pad, F.Cu at (92.4, 68.9)
- added REF**: Pad, clectric-diy:Pad, F.Cu at (110.2, 145.1)
- added REF**: Pad, clectric-diy:Pad, F.Cu at (105.1, 51.1)
- added REF**: Pad, clectric-diy:Pad, F.Cu at (122.8, 117.2)
- added REF**: Pad, clectric-diy:Pad, F.Cu at (130.5, 79.1)
- added REF**: Pad, clectric-diy:Pad, F.Cu at (130.5, 109.6)
- added REF**: Pad, clectric-diy:Pad, F.Cu at (92.4, 114.7)
- added REF**: Pad, clectric-diy:Pad, F.Cu at (130.5, 117.2)
- added REF**: Pad, clectric-diy:Pad, F.Cu at (122.8, 63.9)
- added REF**: Pad, clectric-diy:Pad, F.Cu at (122.8, 132.4)
- added REF**: Pad, clectric-diy:Pad, F.Cu at (87.3, 96.9)
- added REF**: Pad, clectric-diy:Pad, F.Cu at (89.8, 89.2)
- added REF**: Pad, clectric-diy:Pad, F.Cu at (122.8, 109.6)
- added REF**: Pad, clectric-diy:Pad, F.Cu at (94.9, 81.6)
- added REF**: Pad, clectric-diy:Pad, F.Cu at (122.8, 112.1)
- added REF**: Pad, clectric-diy:Pad, F.Cu at (87.3, 91.8)
- added REF**: Pad, clectric-diy:Pad, F.Cu at (127.9, 104.5)
- added REF**: Pad, clectric-diy:Pad, F.Cu at (94.9, 109.6)
- added REF**: Pad, clectric-diy:Pad, F.Cu at (125.4, 117.2)
- added REF**: Pad, clectric-diy:Pad, F.Cu at (130.5, 58.8)
- added REF**: Pad, clectric-diy:Pad, F.Cu at (120.3, 94.3)
- added REF**: Pad, clectric-diy:Pad, F.Cu at (94.9, 63.9)
- added REF**: Pad, clectric-diy:Pad, F.Cu at (84.8, 112.1)
- added REF**: Pad, clectric-diy:Pad, F.Cu at (89.8, 96.9)
- added REF**: Pad, clectric-diy:Pad, F.Cu at (87.3, 107.0)
- added REF**: Pad, clectric-diy:Pad, F.Cu at (92.4, 56.2)
- added REF**: Pad, clectric-diy:Pad, F.Cu at (94.9, 135.0)
- added REF**: Pad, clectric-diy:Pad, F.Cu at (94.9, 99.4)
- added REF**: Pad, clectric-diy:Pad, F.Cu at (122.8, 102.0)
- added REF**: Pad, clectric-diy:Pad, F.Cu at (122.8, 129.9)
- added REF**: Pad, clectric-diy:Pad, F.Cu at (89.8, 117.2)
- added REF**: Pad, clectric-diy:Pad, F.Cu at (89.8, 137.5)
- added REF**: Pad, clectric-diy:Pad, F.Cu at (127.9, 71.5)
- added REF**: Pad, clectric-diy:Pad, F.Cu at (87.3, 79.1)
- moved REF** 125.9 mm to (220.6, 49.4)
- moved REF** 18.7 mm to (110.2, 140.1)
- moved REF** 18.7 mm to (97.5, 140.1)
- moved REF** 18.7 mm to (112.7, 140.1)
- moved REF** 18.7 mm to (107.6, 140.1)
- moved REF** 18.7 mm to (102.5, 140.1)
- moved REF** 18.7 mm to (115.2, 140.1)
- moved REF** 18.7 mm to (97.5, 68.9)
- moved REF** 18.7 mm to (110.2, 68.9)
- moved REF** 18.7 mm to (115.2, 68.9)
- moved REF** 18.7 mm to (112.7, 68.9)
- moved REF** 18.7 mm to (107.6, 68.9)
- moved REF** 18.7 mm to (102.5, 68.9)
- moved REF** 18.7 mm to (107.6, 114.7)
- moved REF** 18.7 mm to (107.6, 102.0)
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Other:
- board size 25 x 100 mm -> 50 x 100 mm
- copper layers 2 -> 4
